File: hardware/if-b01/if-b01.kicad_pcb (KiCad board)
At the start: 4 copper layers, 750 x 400 mm, 90 parts, among them J1 Pico 2 SC1631 left socket, J10 1759114, J11 1759091, J12 1759033, J2 Pico 2 SC1631 right socket, J3 1759033, J4 1759033, J5 1759033, J6 1759033, J7 1759033, J8 1759059, J9 1759059, U1 AM26LV32EIDR, U2 TPL7407LDR, U3 TPL7407LDR

Commit message: Audit fix wave: 35 findings closed across firmware, hardware, CAD, analysis, build definition
Controller (F05/F07/F08/F09/F11/F12/F33): PIO exec-set init with no TX
dependency; strip sequence rewritten with a wire-geometry model rejecting
overlap/wrong-end/loss-of-grip; closure from blade_open_apex/2; length
budget gating so failed correction cannot count; part_clear semantics with
pieces_accepted; commissioning approval interlock; int64 checked jog
arithmetic and per-axis polarity validation. 21/21 machine tests, UBSan
clean.

IF-B01 (F01/F02/F03/F04/F25/F27/F28): J2 physically-correct reversed
footprint + coordinate-derived pin regression; real 1812 SMD PTCs; native
TTL bias network (no 120R terminators); pull-config contract with verified
LOW margin; executable guard-release chain (LADN02 NC blocks, Finder T2,
PLC-RSC R2, fault cases); fuse-coordination honesty; full cabinet budget;
5 V/3 A Siemens identity restored from the maker record.

CAD (F06/F14/F15/F16/F18/F22): second measuring station on the stock side
at X-385 (piece-side proven infeasible for 200 mm parts) with both modules
modeled (550 occurrences) and a position/validity analysis; H006 pattern
collision removed; custom-axis rating constants labelled supplier-stated
with the original 2500/5000 N acceptance restored; stock containment fixed
(F201/M206/M204) with a permanent check; P008 keyed drive boss gives the
payoff brake a real torque path; H007 blade backing carries the cut
reaction with shim-set gap. Payoff shifted 60 mm outboard.

Analysis (F19-F32): full-radius payoff (core 197 N; buffered payoff
selected); driven-contact traction (40-60 N); tension-extension coupling;
thermal design work scoped; throughput/resonance/tooth-pass (79.58 Hz) and
L10 corrections; qualification rejects duplicates with 12-station forces
and provenance; goal matrix rewritten (zero MET; 25 blocked).

Build (F13/F17/F35): one frozen axis config (100 pulses/mm from source);
quantities corrected; portable presets; histor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
Parts:
- removed R1, R2, R3, R4: 120R, IFB01:R_1206_3216
- added C14: 100nF 16V, IFB01:C_0603_1608, F.Cu at (261.0, 116.0)
- added C15: 100nF 16V, IFB01:C_0603_1608, F.Cu at (267.0, 140.0)
- added C16: 100nF 16V, IFB01:C_0603_1608, F.Cu at (273.0, 164.0)
- added C17: 100nF 16V, IFB01:C_0603_1608, F.Cu at (279.0, 188.0)
- added R38: 10k, IFB01:R_0603_1608, F.Cu at (539.5, 164.0)
- added R39: 10k, IFB01:R_0603_1608, F.Cu at (544.5, 188.0)
- added R40: 10k, IFB01:R_0603_1608, F.Cu at (549.5, 212.0)
- added R41: 10k, IFB01:R_0603_1608, F.Cu at (554.5, 92.0)
- added R42: 10k, IFB01:R_0603_1608, F.Cu at (559.5, 116.0)
- added R43: 10k, IFB01:R_0603_1608, F.Cu at (564.5, 140.0)
- added R44: 10k, IFB01:R_0603_1608, F.Cu at (569.5, 164.0)
- added R45: 10k, IFB01:R_0603_1608, F.Cu at (574.5, 188.0)
- added TP10: TP L_ENC_B_N, IFB01:TestPoint_1_0mm, F.Cu at (615.0, 264.0)
- added TP11: TP R_ENC_A_N, IFB01:TestPoint_1_0mm, F.Cu at (619.0, 264.0)
- added TP12: TP R_ENC_B_N, IFB01:TestPoint_1_0mm, F.Cu at (623.0, 264.0)
- added TP9: TP L_ENC_A_N, IFB01:TestPoint_1_0mm, F.Cu at (611.0, 264.0)
- F1: value MF-R050 -> MF-MSMF050/60X
- F2, F3: value MF-R050 -> MF-MSMF050/16X
- J2: footprint IFB01:PICO_SOCKET_1X20 -> IFB01:PICO_SOCKET_1X20_RIGHT
- moved U3 463.9 mm to (192.0, 260.0)
- moved D1 99.0 mm to (285.0, 212.0)
- moved D6 99.0 mm to (315.0, 188.0)
- moved D7 99.0 mm to (321.0, 212.0)
- moved F2 99.0 mm to (357.0, 188.0)
- moved F3 99.0 mm to (367.0, 212.0)
- moved D10 53.7 mm to (339.0, 140.0)
- moved D2 53.7 mm to (291.0, 92.0)
- moved D3 53.7 mm to (297.0, 116.0)
- moved D4 53.7 mm to (303.0, 140.0)
- moved D5 53.7 mm to (309.0, 164.0)
- moved D8 53.7 mm to (327.0, 92.0)
- moved D9 53.7 mm to (333.0, 116.0)
- moved F1 53.7 mm to (347.0, 164.0)
- moved U1 52.0 mm to (637.0, 212.0)
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Routing:
- net /0V_PELV: track 9829.4 -> 10508.4 mm, vias 116 -> 132
- net /R_ENC_A_N: track 967.0 -> 1633.4 mm, vias 6 -> 12
- net /L_ENC_B_N: track 1019.1 -> 1624.5 mm, vias 6 -> 12
- net /R_ENC_B_N: track 945.9 -> 1523.2 mm, vias 6 -> 12
- net /BUZZER_NEG: track 961.6 -> 384.7 mm
- net /RED_NEG: track 1078.0 -> 508.2 mm
- net /GREEN_NEG: track 1054.3 -> 484.5 mm
- net /FR_DIR_NEG: track 1023.8 -> 462.0 mm
- net /L_ENC_A_N: track 1055.9 -> 1606.3 mm, vias 6 -> 12
- net /L_ENC_A_P: track 1069.3 -> 576.1 mm, vias 6 -> 4
- net /L_ENC_B_P: track 1033.0 -> 572.9 mm, vias 6 -> 4
- net /R_ENC_A_P: track 982.9 -> 535.4 mm, vias 6 -> 4
- net /R_ENC_B_P: track 957.2 -> 534.3 mm, vias 6 -> 4
- net /+5V_ENC_R: track 804.6 -> 986.0 mm, vias 4 -> 8
- net /DRV_ENA_NEG: track 1785.3 -> 1604.8 mm
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