File: hardware/if-b01/if-b01.kicad_sch (KiCad schematic)
At the start: 100 parts, among them J1 Pico 2 SC1631 left socket, J10 1759114, J11 1759091, J12 1759033, J2 Pico 2 SC1631 right socket, J3 1759033, J4 1759033, J5 1759033, J6 1759033, J7 1759033, J8 1759059, J9 1759059, P10 1757314, P11 1757291, P12 1757233, P3 1757233, P4 1757233, P5 1757233, P6 1757233, P7 1757233, P8 1757259, P9 1757259, U1 AM26LV32EIDR, U2 TPL7407LDR, U3 TPL7407LDR

Commit message: Audit fix wave: 35 findings closed across firmware, hardware, CAD, analysis, build definition
Controller (F05/F07/F08/F09/F11/F12/F33): PIO exec-set init with no TX
dependency; strip sequence rewritten with a wire-geometry model rejecting
overlap/wrong-end/loss-of-grip; closure from blade_open_apex/2; length
budget gating so failed correction cannot count; part_clear semantics with
pieces_accepted; commissioning approval interlock; int64 checked jog
arithmetic and per-axis polarity validation. 21/21 machine tests, UBSan
clean.

IF-B01 (F01/F02/F03/F04/F25/F27/F28): J2 physically-correct reversed
footprint + coordinate-derived pin regression; real 1812 SMD PTCs; native
TTL bias network (no 120R terminators); pull-config contract with verified
LOW margin; executable guard-release chain (LADN02 NC blocks, Finder T2,
PLC-RSC R2, fault cases); fuse-coordination honesty; full cabinet budget;
5 V/3 A Siemens identity restored from the maker record.

CAD (F06/F14/F15/F16/F18/F22): second measuring station on the stock side
at X-385 (piece-side proven infeasible for 200 mm parts) with both modules
modeled (550 occurrences) and a position/validity analysis; H006 pattern
collision removed; custom-axis rating constants labelled supplier-stated
with the original 2500/5000 N acceptance restored; stock containment fixed
(F201/M206/M204) with a permanent check; P008 keyed drive boss gives the
payoff brake a real torque path; H007 blade backing carries the cut
reaction with shim-set gap. Payoff shifted 60 mm outboard.

Analysis (F19-F32): full-radius payoff (core 197 N; buffered payoff
selected); driven-contact traction (40-60 N); tension-extension coupling;
thermal design work scoped; throughput/resonance/tooth-pass (79.58 Hz) and
L10 corrections; qualification rejects duplicates with 12-station forces
and provenance; goal matrix rewritten (zero MET; 25 blocked).

Build (F13/F17/F35): one frozen axis config (100 pulses/mm from source);
quantities corrected; portable presets; histor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
Parts:
- removed R1, R2, R3, R4: 120R, IFB01:R_1206_3216, symbol IFB01:R
- added C14, C15, C16, C17: 100nF 16V, IFB01:C_0603_1608, symbol IFB01:C
- added R38, R39, R40, R41, R42, R43, R44, R45: 10k, IFB01:R_0603_1608, symbol IFB01:R
- added TP10: TP L_ENC_B_N, IFB01:TestPoint_1_0mm, symbol IFB01:TP
- added TP11: TP R_ENC_A_N, IFB01:TestPoint_1_0mm, symbol IFB01:TP
- added TP12: TP R_ENC_B_N, IFB01:TestPoint_1_0mm, symbol IFB01:TP
- added TP9: TP L_ENC_A_N, IFB01:TestPoint_1_0mm, symbol IFB01:TP
- F1: value MF-R050 -> MF-MSMF050/60X; MPN MF-R050 -> MF-MSMF050/60X
- F2, F3: value MF-R050 -> MF-MSMF050/16X; MPN MF-R050 -> MF-MSMF050/16X
- J2: footprint IFB01:PICO_SOCKET_1X20 -> IFB01:PICO_SOCKET_1X20_RIGHT
Connections:
- net +5V_ENC_L: now also R38.1, R40.1
- net +5V_ENC_R: now also R42.1, R44.1
- net 0V_PELV: now also C14.2, C15.2, C16.2, C17.2, R39.1, R41.1, R43.1, R45.1
- net L_ENC_A_N: now also C14.1, R38.2, R39.2, TP9.1 (TP)
- net L_ENC_B_N: now also C15.1, R40.2, R41.2, TP10.1 (TP)
- net R_ENC_A_N: now also C16.1, R42.2, R43.2, TP11.1 (TP)
- net R_ENC_B_N: now also C17.1, R44.2, R45.2, TP12.1 (TP)
Other:
- note added: "J8/J9 RU3100 single-ended TTL (TTL mode selected via IO-Link): encoder A/B drive J8/J9 pins 3/5 (A+/B+); A-/B- (pins 4/6) are held at the 2.5 V mid-bias by R38-R45 10k 1 % and C14-C17 100 nF; the R1-R4 120 ohm differential terminators are removed."
- note added: "PULL-CONFIG CONTRACT: RP2350 internal pull-up/-down MUST be disabled in BOTH firmware images on GP12 GP13 GP14 GP15 GP16 GP27 GP18 GP19 GP20 GP21; the only pull on each dry-contact pin is the board external 47k 1 % pull-up to 3V3_MCU. Nominal LOW = 3.3 V x 10k / (10k + 47k) = 0.579 V < VIL max 0.8 V."
